Commit message: PR06: reproduce incorrect lidar parent

File: src/course_description/urdf/ackerman_robot.urdf.xacro (robot description, xacro)
@@ -210,5 +210,5 @@
   </joint>
   <joint name="lidar_joint" type="fixed">
-    <parent link="base_link"/>
+    <parent link="camera_link"/>
     <child link="lidar_link"/>
     <origin xyz="${sensor_x} 0 ${sensor_z}" rpy="0 0 0"/>

Commit message: PR06: restore correct lidar parent

File: src/course_description/urdf/ackerman_robot.urdf.xacro (robot description, xacro)
@@ -210,5 +210,5 @@
   </joint>
   <joint name="lidar_joint" type="fixed">
-    <parent link="camera_link"/>
+    <parent link="base_link"/>
     <child link="lidar_link"/>
     <origin xyz="${sensor_x} 0 ${sensor_z}" rpy="0 0 0"/>
